File: New_Clock/Infinity Mirror/Infinity Mirror.brd (EAGLE design)
At the start: 100 x 80 mm, 2 parts

Commit message: board files almost complete
Parts:
- removed U$2: DS1307, Infinity Mirror:SOIC_8
- added B1: CR1220, microbuilder:CR1220
- added C1: 0.1uF, microbuilder:0805-NO
- added C2, C3, C4, C5: (no value), Terra_4.0_12_DIP_JJM_EB2_9-6-2018d:SPARKFUN-CAPACITORS_0805
- added IC1: MSGEQ7P, SparkFun-IC-Special-Function:DIP08
- added J1: (no value), RC1a_Main_2-20-2018_m:SPARKFUN-CONNECTORS_1X02_LOCK
- added J2: (no value), SparkFun-Connectors:1X06
- added J3: (no value), SparkFun-Connectors:1X03
- added Q1: 32.768, microbuilder:CRYSTAL_8X3.8
- added R1, R2: 10K, microbuilder:0805-NO
- added R3, R5: (no value), RC1a_Main_2-20-2018_m:SPARKFUN-PASSIVES_0805
- added U1: DS1307, microbuilder:SOIC8_150MIL
- U$1: value ARDUINO_PROTRINKET_5V -> ADAFRUIT_PRO_TRINKET_NO-DIMENSION; device _111_IH:ARDUINO_PROTRINKET_5V -> _111_IH:ARDUINO_PRO_TRINKET_5V_NO-DIMENSION
- moved U$1 99.3 mm to (77.0, 13.0), turned to 90 degrees
Connections:
- new net 3-OUT: IC1.3, U$1.TA3
- new net 4-STROBE: IC1.4, U$1.T8
- new net 6: C4.1, IC1.6
- new net 7-RESET: IC1.7, U$1.T~10
- new net AUDIO_IN: C2.1, IC1.5
- new net ELECTRET_AUDIO_OUT: J2.3, R3.2
- new net GND: B1.-, C1.2, C3.2, C4.2, C5.1, IC1.2, J1.2, J2.1, J3.1, U$1.TG, U1.4
- new net N$2: J3.2
- new net N$5: C3.1, IC1.8, R5.1
- new net N$8: C2.2, R3.1
- new net POT_1: J2.6, U$1.TA0
- new net POT_2: J2.5, U$1.TA1
- new net POT_3: J2.4, U$1.TA2
- new net SCL: R2.2, U$1.TA5, U1.6
- new net SDA: R1.1, U$1.TA4, U1.5
- new net SQW: U1.7
- new net VBAT: B1.+$1, U1.3
- new net VCC: C1.1, C5.2, IC1.1, J1.1, J2.2, J3.3, R1.2, R2.1, R5.2, U$1.TBAT+, U1.8
- new net XI: Q1.P$1, U1.1
- new net XO: Q1.P$4, U1.2
Routing:
- net VCC: track 0.00 -> 154.2 mm
- net 3-OUT: track 0.00 -> 80.0 mm
- net 7-RESET: track 0.00 -> 75.4 mm
- net POT_3: track 0.00 -> 57.0 mm
- net 4-STROBE: track 0.00 -> 54.1 mm
- net POT_2: track 0.00 -> 51.4 mm
- net POT_1: track 0.00 -> 44.9 mm
- net SDA: track 0.00 -> 28.1 mm
- net SCL: track 0.00 -> 22.0 mm
- net VBAT: track 0.00 -> 18.8 mm
- net AUDIO_IN: track 0.00 -> 7.76 mm
- net 6: track 0.00 -> 6.99 mm
- net N$5: track 0.00 -> 6.09 mm
- net XO: track 0.00 -> 4.91 mm
- net N$8: track 0.00 -> 4.80 mm
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- added copper zone on layer 1, net GND
Other:
- board size 100 x 80 mm -> 81 x 26 mm

Commit message: finished pcb rough draft and BoM
Parts:
- removed Q1: 32.768, microbuilder:CRYSTAL_8X3.8
- added J4: LED_CAP, RC1a_Main_2-20-2018_m:SPARKFUN-CONNECTORS_1X02_LOCK
- added R4: 220, RC1a_Main_2-20-2018_m:SPARKFUN-PASSIVES_0805
- added S1: (no value), SparkFun-Switches:SWITCH_SPDT_PTH_11.6X4.0MM_LOCK
- added Y1: 32.768kHz, SparkFun-Clocks:CRYSTAL-PTH-2X6-CYL
- C2: value (none) -> 0.01uF
- C3: value (none) -> 33pF; device Terra_4.0_12_DIP_JJM_EB2_9-6-2018d:SPARKFUN-CAPACITORS_0805 -> SparkFun-Capacitors:0805
- C4, C5: value (none) -> 0.1uF
- J1: value (none) -> Vsupply
- J3: value (none) -> LED
- R3: value (none) -> 22k
- R5: value (none) -> 200k
- moved J3 24.0 mm to (3.03, 24.0), turned to 270 degrees
- moved B1 5.10 mm to (34.0, 7.00)
- moved R2 4.57 mm to (69.4, 8.73)
- moved C1 4.22 mm to (65.6, 8.73)
- moved C2 4.16 mm to (13.5, 8.11), turned to 0 degrees
- moved R3 2.28 mm to (16.6, 6.93)
- moved J1 1.88 mm to (47.0, 7.35), turned to 270 degrees
- moved IC1 0.59 mm to (14.6, 13.8)
- moved C5 0.54 mm to (17.2, 19.4)
- moved C4 0.19 mm to (8.44, 9.44)
- moved R1 0.18 mm to (69.8, 15.0)
Connections:
- net 6 renamed 6-GND
- net N$2 renamed DATA_OUT
- net N$5 renamed 8-CKIN
- new net 3: R4.2, S1.2
- new net ~3: R4.1, U$1.T~3
- net GND: now also J4.2, S1.3
- net VCC: now also J4.1, S1.1
- net XI: now also Y1.2; no longer Q1.P$1
- net XO: now also Y1.1; no longer Q1.P$4
Routing:
- net ~3: track 0.00 -> 20.8 mm
- net 3: track 0.00 -> 10.2 mm
- net 3-OUT: track 80.0 -> 74.0 mm
- net VCC: track 154.2 -> 159.8 mm, vias 0 -> 1
- net AUDIO_IN: track 7.76 -> 3.29 mm
- net SDA: track 28.1 -> 31.0 mm
- net GND: track 1.88 -> 4.49 mm
- net N$8: track 4.80 -> 2.42 mm
- net XO: track 4.91 -> 6.95 mm
- net VBAT: track 18.8 -> 20.4 mm
- net POT_3: track 57.0 -> 58.4 mm
- net ELECTRET_AUDIO_OUT: track 2.76 -> 4.13 mm
- net POT_1: track 44.9 -> 46.1 mm
- net POT_2: track 51.4 -> 52.5 mm
- added copper zone on layer 16, net GND
Other:
- outline, holes or cut-outs redrawn

Commit message: fixed errors in infinity mirror draft. This one is ordered, hopefully it works :D
Parts:
- J2: value (none) -> AUDIO_POTS
- moved C1 8.29 mm to (65.0, 17.0)
- moved R2 2.00 mm to (71.4, 8.73)
Routing:
- net VCC: track 159.8 -> 164.3 mm, vias 1 -> 3
- net XO: track 6.95 -> 4.95 mm
- net GND: track 4.49 -> 5.82 mm
- removed copper zone on layer 16, net GND
