File: New_Clock/Infinity Mirror/Infinity Mirror.sch (EAGLE design)
At the start: 2 parts

Commit message: board files almost complete
Parts:
- removed U$2: DS1307, Infinity Mirror:DS1307
- added B1: CR1220, microbuilder:BATTERYCR1220_SMT
- added C1: 0.1uF, microbuilder:CAP_CERAMIC0805-NOOUTLINE
- added C2, C3, C4, C5: (no value), Terra_4.0_12_DIP_JJM_EB2_9-6-2018d:SPARKFUN-CAPACITORS_CAP0805
- added IC1: MSGEQ7P, SparkFun-IC-Special-Function:MSGEQ7DIL
- added J1: (no value), RC1a_Main_2-20-2018_m:SPARKFUN-CONNECTORS_CONN_02LOCK
- added J2: (no value), SparkFun-Connectors:CONN_06SILK_FEMALE_PTH
- added J3: (no value), SparkFun-Connectors:CONN_03
- added Q1: 32.768, microbuilder:CRYSTAL8.0X3.8
- added R1, R2: 10K, microbuilder:RESISTOR0805_NOOUTLINE
- added R3, R5: (no value), RC1a_Main_2-20-2018_m:SPARKFUN-PASSIVES_RESISTOR0805-RES
- added U1: DS1307, microbuilder:RTC_DS1307
- U$1: value ARDUINO_PROTRINKET_5V -> ADAFRUIT_PRO_TRINKET_NO-DIMENSION; device _111_IH:ARDUINO_PROTRINKET_5V -> _111_IH:ADAFRUIT_PRO_TRINKET_NO-DIMENSION
Connections:
- new net 3-OUT: IC1.3-OUT, U$1.A3
- new net 4-STROBE: IC1.4-STROBE, U$1.8
- new net 6: C4.1, IC1.6-GND
- new net 7-RESET: IC1.7-RESET, U$1.~10
- new net AUDIO_IN: C2.1, IC1.5-IN
- new net ELECTRET_AUDIO_OUT: J2.3, R3.2
- new net GND: B1.-, C1.2, C3.2, C4.2, C5.1, IC1.2-VSSA, J1.2, J2.1, J3.1, U$1.G, U1.GND
- new net N$2: J3.2
- new net N$5: C3.1, IC1.8-CKIN, R5.1
- new net N$8: C2.2, R3.1
- new net POT_1: J2.6, U$1.A0
- new net POT_2: J2.5, U$1.A1
- new net POT_3: J2.4, U$1.A2
- new net SCL: R2.2, U$1.A5, U1.SCL
- new net SDA: R1.1, U$1.A4, U1.SDA
- new net SQW: U1.SQW/OUT
- new net VBAT: B1.+, U1.VBAT
- new net VCC: C1.1, C5.2, IC1.1-VDD, J1.1, J2.2, J3.3, R1.2, R2.1, R5.2, U$1.BAT+, U1.VCC
- new net XI: Q1.1, U1.X1
- new net XO: Q1.2, U1.X2

Commit message: finished pcb rough draft and BoM
Parts:
- removed Q1: 32.768, microbuilder:CRYSTAL8.0X3.8
- added J4: LED_CAP, RC1a_Main_2-20-2018_m:SPARKFUN-CONNECTORS_CONN_02LOCK
- added R4: 220, RC1a_Main_2-20-2018_m:SPARKFUN-PASSIVES_RESISTOR0805-RES
- added S1: (no value), SparkFun-Switches:SWITCH-SPDT-PTH-11.6X4.0MM-LOCK
- added Y1: 32.768kHz, SparkFun-Clocks:CRYSTAL-32.768KHZPTH-2X6
- C2: value (none) -> 0.01uF
- C3: value (none) -> 33pF; device Terra_4.0_12_DIP_JJM_EB2_9-6-2018d:SPARKFUN-CAPACITORS_CAP0805 -> SparkFun-Capacitors:0.33UF/330NF-0805-50V-10%
- C4, C5: value (none) -> 0.1uF
- J1: value (none) -> Vsupply
- J3: value (none) -> LED
- R3: value (none) -> 22k
- R5: value (none) -> 200k
Connections:
- net 6 renamed 6-GND
- net N$2 renamed DATA_OUT
- net N$5 renamed 8-CKIN
- new net 3: R4.2, S1.P
- new net ~3: R4.1, U$1.~3
- net GND: now also J4.2, S1.S
- net VCC: now also J4.1, S1.O
- net XI: now also Y1.2; no longer Q1.1
- net XO: now also Y1.1; no longer Q1.2
Other:
- moved on the sheet: C2, C3, R3, R5

Commit message: fixed errors in infinity mirror draft. This one is ordered, hopefully it works :D
Parts:
- J2: value (none) -> AUDIO_POTS
Changed lines of the file:
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@@
 <part name="R3" library="RC1a_Main_2-20-2018_m" deviceset="SPARKFUN-PASSIVES_RESISTOR" device="0805-RES" value="22k"/>
 <part name="C2" library="Terra_4.0_12_DIP_JJM_EB2_9-6-2018d" deviceset="SPARKFUN-CAPACITORS_CAP" device="0805" value="0.01uF"/>
-<part name="J2" library="SparkFun-Connectors" library_urn="urn:adsk.eagle:library:513" deviceset="CONN_06" device="SILK_FEMALE_PTH" package3d_urn="urn:adsk.eagle:package:38009/1"/>
+<part name="J2" library="SparkFun-Connectors" library_urn="urn:adsk.eagle:library:513" deviceset="CONN_06" device="SILK_FEMALE_PTH" package3d_urn="urn:adsk.eagle:package:38009/1" value="AUDIO_POTS"/>
 <part name="GND3" library="supply1" library_urn="urn:adsk.eagle:library:371" deviceset="GND" device=""/>
 <part name="R5" library="RC1a_Main_2-20-2018_m" deviceset="SPARKFUN-PASSIVES_RESISTOR" device="0805-RES" value="200k"/>
@@
 <pinref part="IC1" gate="G$1" pin="1-VDD"/>
 <pinref part="P+5" gate="VCC" pin="VCC"/>
-<wire x1="50.8" y1="83.82" x2="55.88" y2="83.82" width="0.1524" layer="91"/>
+<wire x1="50.8" y1="83.82" x2="58.42" y2="83.82" width="0.1524" layer="91"/>
 <pinref part="C5" gate="G$1" pin="2"/>
-<wire x1="55.88" y1="83.82" x2="58.42" y2="83.82" width="0.1524" layer="91"/>
-<wire x1="58.42" y1="83.82" x2="60.96" y2="83.82" width="0.1524" layer="91"/>
-<wire x1="60.96" y1="83.82" x2="60.96" y2="91.44" width="0.1524" layer="91"/>
+<wire x1="58.42" y1="83.82" x2="60.96" y2="86.36" width="0.1524" layer="91"/>
+<wire x1="60.96" y1="86.36" x2="60.96" y2="91.44" width="0.1524" layer="91"/>
 <label x="55.88" y="83.82" size="1.778" layer="95"/>
+<junction x="58.42" y="83.82"/>
 </segment>
 </net>
