File: PCB/infinity_mirror_proj_d/infinity_mirror_revd.sch (EAGLE design)
At the start: 35 parts, among them J1 POWER_JACKPTH_BREAD, Q1 800mA/40V, Q2 800mA/40V, Q3 BSS138, U1 3.3LDO

Commit message: pcb refactor
Parts:
- J2: value (none) -> CAP
- J3: value (none) -> SERIAL
Connections:
- removed net N$1: J2.2
- net DTR: now also J3.4; no longer J3.2
- net GND: now also J2.2
- net U0RXD: now also J3.2; no longer J3.4
Changed lines of the file:
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@@
 <?xml version="1.0" encoding="utf-8"?>
 <!DOCTYPE eagle SYSTEM "eagle.dtd">
-<eagle version="9.3.0">
+<eagle version="9.6.2">
 <drawing>
 <settings>
@@
 <part name="GND12" library="supply1" library_urn="urn:adsk.eagle:library:371" deviceset="GND" device=""/>
 <part name="GND13" library="supply1" library_urn="urn:adsk.eagle:library:371" deviceset="GND" device=""/>
-<part name="J3" library="SparkFun-Connectors" deviceset="CONN_04" device=""/>
-<part name="J2" library="SparkFun-Connectors" deviceset="CONN_02" device=""/>
+<part name="J3" library="SparkFun-Connectors" deviceset="CONN_04" device="" value="SERIAL"/>
+<part name="J2" library="SparkFun-Connectors" deviceset="CONN_02" device="" value="CAP"/>
 </parts>
 <sheets>
@@
 <pinref part="U$2" gate="G$1" pin="P$2"/>
 <label x="73.66" y="5.08" size="1.778" layer="95"/>
-<wire x1="55.88" y1="7.606" x2="55.88" y2="5.08" width="0.1524" layer="91"/>
 <wire x1="55.88" y1="5.08" x2="81.28" y2="5.08" width="0.1524" layer="91"/>
 <pinref part="GND9" gate="1" pin="GND"/>
 <wire x1="55.88" y1="0" x2="55.88" y2="5.08" width="0.1524" layer="91"/>
+<pinref part="J2" gate="G$1" pin="2"/>
+<wire x1="55.88" y1="5.08" x2="55.88" y2="10.16" width="0.1524" layer="91"/>
 <junction x="55.88" y="5.08"/>
 </segment>
@@
 </segment>
 <segment>
-<pinref part="J3" gate="G$1" pin="4"/>
-<wire x1="-96.52" y1="-71.12" x2="-88.9" y2="-71.12" width="0.1524" layer="91"/>
-<label x="-93.98" y="-71.12" size="1.778" layer="95"/>
+<pinref part="J3" gate="G$1" pin="2"/>
+<wire x1="-96.52" y1="-76.2" x2="-88.9" y2="-76.2" width="0.1524" layer="91"/>
+<label x="-93.98" y="-76.2" size="1.778" layer="95"/>
 </segment>
 </net>
@@
 </segment>
 <segment>
-<pinref part="J3" gate="G$1" pin="2"/>
-<wire x1="-96.52" y1="-76.2" x2="-88.9" y2="-76.2" width="0.1524" layer="91"/>
-<label x="-93.98" y="-76.2" size="1.778" layer="95"/>
+<pinref part="J3" gate="G$1" pin="4"/>
+<wire x1="-96.52" y1="-71.12" x2="-88.9" y2="-71.12" width="0.1524" layer="91"/>
+<label x="-93.98" y="-71.12" size="1.778" layer="95"/>
 </segment>
 </net>
@@
 </segment>
 </net>
-<net name="N$1" class="0">
-<segment>
-<pinref part="J2" gate="G$1" pin="2"/>
-<wire x1="55.88" y1="10.16" x2="55.88" y2="7.62" width="0.1524" layer="91"/>
-</segment>
-</net>
