File: PCB/infinity_mirror_proj_g/infinity_mirror_rev_g.sch (EAGLE design)
At the start: 31 parts, among them J1 POWER_JACKPTH_BREAD, J2 LED_CAP, J3 SERIAL, Q3 BSS138, U1 3.3LDO

Commit message: serial connector from 4pin to 3pin. changed led data gpio to reduce trace length
Parts:
- J3: device SparkFun-Connectors:CONN_04 -> SparkFun-Connectors:CONN_03
Connections:
- removed net IO23: Q3.S, R10.1, U$1.GPIO23
- new net IO33: Q3.S, R10.1, U$1.GPIO33
- net VCC_2: no longer J3.4
Changed lines of the file:
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@@
 <part name="GND12" library="supply1" library_urn="urn:adsk.eagle:library:371" deviceset="GND" device=""/>
 <part name="GND13" library="supply1" library_urn="urn:adsk.eagle:library:371" deviceset="GND" device=""/>
-<part name="J3" library="SparkFun-Connectors" library_urn="urn:adsk.eagle:library:513" deviceset="CONN_04" device="" package3d_urn="urn:adsk.eagle:package:38085/1" value="SERIAL"/>
+<part name="J3" library="SparkFun-Connectors" library_urn="urn:adsk.eagle:library:513" deviceset="CONN_03" device="" package3d_urn="urn:adsk.eagle:package:38063/1" value="SERIAL"/>
 <part name="J2" library="SparkFun-Connectors" deviceset="CONN_02" device="" value="LED_CAP"/>
 <part name="U$1" library="infinity_mirror_revd" deviceset="ESP32-WROOM-32E" device=""/>
@@
 <wire x1="0" y1="-101.6" x2="0" y2="-50.8" width="0.1524" layer="97"/>
 <wire x1="0" y1="-50.8" x2="114.3" y2="-50.8" width="0.1524" layer="97"/>
-<wire x1="-2.54" y1="-50.8" x2="-93.98" y2="-50.8" width="0.1524" layer="97"/>
-<wire x1="-93.98" y1="-50.8" x2="-93.98" y2="-101.6" width="0.1524" layer="97"/>
-<wire x1="-93.98" y1="-101.6" x2="-2.54" y2="-101.6" width="0.1524" layer="97"/>
+<wire x1="-2.54" y1="-50.8" x2="-96.52" y2="-50.8" width="0.1524" layer="97"/>
+<wire x1="-96.52" y1="-50.8" x2="-96.52" y2="-101.6" width="0.1524" layer="97"/>
+<wire x1="-96.52" y1="-101.6" x2="-2.54" y2="-101.6" width="0.1524" layer="97"/>
 <wire x1="-2.54" y1="-101.6" x2="-2.54" y2="-50.8" width="0.1524" layer="97"/>
 <text x="48.26" y="119.38" size="1.778" layer="97">ROTARY ENCODER</text>
@@
 <attribute name="VALUE" x="-38.1" y="-86.36" size="1.778" layer="96"/>
 </instance>
-<instance part="J3" gate="G$1" x="-86.36" y="-73.66" smashed="yes">
-<attribute name="VALUE" x="-91.44" y="-81.026" size="1.778" layer="96" font="vector"/>
-<attribute name="NAME" x="-91.44" y="-65.532" size="1.778" layer="95" font="vector"/>
+<instance part="J3" gate="J$1" x="-88.9" y="-73.66" smashed="yes">
+<attribute name="VALUE" x="-93.98" y="-81.026" size="1.778" layer="96" font="vector"/>
+<attribute name="NAME" x="-93.98" y="-65.532" size="1.778" layer="95" font="vector"/>
 </instance>
 <instance part="J2" gate="G$1" x="63.5" y="12.7" smashed="yes" rot="R180">
@@
 </segment>
 <segment>
-<pinref part="J3" gate="G$1" pin="3"/>
+<pinref part="J3" gate="J$1" pin="3"/>
 <wire x1="-81.28" y1="-71.12" x2="-76.2" y2="-71.12" width="0.1524" layer="91"/>
 <label x="-81.28" y="-71.12" size="1.778" layer="95"/>
@@
 <pinref part="U$1" gate="G$1" pin="GND@3"/>
 <wire x1="25.4" y1="22.86" x2="33.02" y2="22.86" width="0.1524" layer="91"/>
-<label x="27.94" y="22.86" size="1.778" layer="95"/>
-</segment>
-<segment>
-<pinref part="J3" gate="G$1" pin="1"/>
+<label x="30.48" y="22.86" size="1.778" layer="95"/>
+</segment>
+<segment>
+<pinref part="J3" gate="J$1" pin="1"/>
 <wire x1="-81.28" y1="-76.2" x2="-76.2" y2="-76.2" width="0.1524" layer="91"/>
 <label x="-81.28" y="-76.2" size="1.778" layer="95"/>
@@
 </segment>
 <segment>
-<pinref part="J3" gate="G$1" pin="2"/>
+<pinref part="J3" gate="J$1" pin="2"/>
 <wire x1="-81.28" y1="-73.66" x2="-76.2" y2="-73.66" width="0.1524" layer="91"/>
 <label x="-81.28" y="-73.66" size="1.778" layer="95"/>
@@
 <pinref part="U$1" gate="G$1" pin="GPIO0"/>
 <wire x1="25.4" y1="-10.16" x2="38.1" y2="-10.16" width="0.1524" layer="91"/>
-<label x="27.94" y="-10.16" size="1.778" layer="95"/>
+<label x="30.48" y="-10.16" size="1.778" layer="95"/>
 </segment>
 </net>
@@
 <junction x="55.88" y="-35.56"/>
 </segment>
-<segment>
-<pinref part="J3" gate="G$1" pin="4"/>
-<wire x1="-81.28" y1="-68.58" x2="-76.2" y2="-68.58" width="0.1524" layer="91"/>
-<label x="-81.28" y="-68.58" size="1.778" layer="95"/>
-</segment>
 </net>
 <net name="VCC_1" class="0">
@@
 <segment>
 <pinref part="U$1" gate="G$1" pin="GPIO25"/>
-<wire x1="-27.94" y1="0" x2="-33.02" y2="0" width="0.1524" layer="91"/>
-<label x="-38.1" y="0" size="1.778" layer="95"/>
+<wire x1="-27.94" y1="0" x2="-40.64" y2="0" width="0.1524" layer="91"/>
+<label x="-40.64" y="0" size="1.778" layer="95"/>
 </segment>
 </net>
@@
 </segment>
 </net>
-<net name="IO23" class="0">
-<segment>
-<pinref part="Q3" gate="NMOS" pin="S"/>
-<wire x1="81.28" y1="-33.02" x2="81.28" y2="-35.56" width="0.1524" layer="91"/>
-<wire x1="81.28" y1="-35.56" x2="81.28" y2="-43.18" width="0.1524" layer="91"/>
-<junction x="81.28" y="-35.56"/>
-<wire x1="81.28" y1="-35.56" x2="71.12" y2="-35.56" width="0.1524" layer="91"/>
-<pinref part="R10" gate="G$1" pin="1"/>
-<label x="83.82" y="-43.18" size="1.778" layer="95" rot="R90"/>
-</segment>
-<segment>
-<pinref part="U$1" gate="G$1" pin="GPIO23"/>
-<wire x1="25.4" y1="20.32" x2="33.02" y2="20.32" width="0.1524" layer="91"/>
-<label x="27.94" y="20.32" size="1.778" layer="95"/>
-</segment>
-</net>
 <net name="EN" class="0">
 <segment>
@@
 <wire x1="-43.18" y1="5.08" x2="-50.8" y2="5.08" width="0.1524" layer="91"/>
 <junction x="-50.8" y="5.08"/>
-<label x="-33.02" y="17.78" size="1.778" layer="95"/>
+<label x="-35.56" y="17.78" size="1.778" layer="95"/>
 <pinref part="U$1" gate="G$1" pin="EN"/>
 <wire x1="-43.18" y1="5.08" x2="-43.18" y2="17.78" width="0.1524" layer="91"/>
@@
 </segment>
 </net>
+<net name="IO33" class="0">
+<segment>
+<pinref part="U$1" gate="G$1" pin="GPIO33"/>
+<wire x1="-27.94" y1="2.54" x2="-38.1" y2="2.54" width="0.1524" layer="91"/>
+<label x="-38.1" y="2.54" size="1.778" layer="95"/>
+</segment>
+<segment>
+<pinref part="Q3" gate="NMOS" pin="S"/>
+<wire x1="81.28" y1="-33.02" x2="81.28" y2="-35.56" width="0.1524" layer="91"/>
+<wire x1="81.28" y1="-35.56" x2="81.28" y2="-43.18" width="0.1524" layer="91"/>
+<junction x="81.28" y="-35.56"/>
+<wire x1="81.28" y1="-35.56" x2="71.12" y2="-35.56" width="0.1524" layer="91"/>
+<pinref part="R10" gate="G$1" pin="1"/>
+<label x="83.82" y="-43.18" size="1.778" layer="95" rot="R90"/>
+</segment>
+</net>
